Commit message: raess1

File: robot_gym/util/pybullet_data/robots/k3lso.urdf (robot description, URDF)
Before this commit: robot k3lso_robot, 17 links, 16 joints
Links:
- link abduct_fl_1: geometry collision mesh filename=k3lso/obj/abduct_fl_1.obj scale=0.001 0.001 0.001; visual mesh filename=k3lso/obj/abduct_fl_1.obj scale=0.001 0.001 0.001
- link abduct_fr_1: geometry collision mesh filename=k3lso/obj/abduct_fr_1.obj scale=0.001 0.001 0.001; visual mesh filename=k3lso/abduct_fr_1.stl scale=0.001 0.001 0.001
- link abduct_hl_1: geometry collision mesh filename=k3lso/obj/abduct_hl_1.obj scale=0.001 0.001 0.001; visual mesh filename=k3lso/obj/abduct_hl_1.obj scale=0.001 0.001 0.001
- link abduct_hr_1: geometry collision mesh filename=k3lso/obj/abduct_hr_1.obj/ scale=0.001 0.001 0.001; visual mesh filename=k3lso/obj/abduct_hr_1.obj scale=0.001 0.001 0.001
- link base_link: geometry collision mesh filename=k3lso/obj/base_link.obj scale=0.001 0.001 0.001; visual mesh filename=k3lso/base_link.stl scale=0.001 0.001 0.001
- link shank_hl_1: geometry collision mesh filename=k3lso/obj/shank_hl_1.obj scale=0.001 0.001 0.001; visual mesh filename=k3lso/obj/shank_hl_1.obj scale=0.001 0.001 0.001
- link shank_hl_2: geometry collision mesh filename=k3lso/obj/shank_hl_2.obj scale=0.001 0.001 0.001; visual mesh filename=k3lso/obj/shank_hl_2.obj scale=0.001 0.001 0.001
- link shank_hl_3: geometry collision mesh filename=k3lso/obj/shank_hl_3.obj scale=0.001 0.001 0.001; visual mesh filename=k3lso/obj/shank_hl_3.obj scale=0.001 0.001 0.001
- link shank_hl_4: geometry collision mesh filename=k3lso/obj/shank_hl_4.obj scale=0.001 0.001 0.001; visual mesh filename=k3lso/obj/shank_hl_4.obj scale=0.001 0.001 0.001
- link thigh_hl_1: geometry collision mesh filename=k3lso/obj/thigh_hl_1.obj scale=0.001 0.001 0.001; visual mesh filename=k3lso/obj/thigh_hl_1.obj scale=0.001 0.001 0.001
- link thigh_hl_2: geometry collision mesh filename=k3lso/obj/thigh_hl_2.obj scale=0.001 0.001 0.001; visual mesh filename=k3lso/obj/thigh_hl_2.obj scale=0.001 0.001 0.001
- link thigh_hr_1: geometry collision mesh filename=k3lso/obj/thigh_hr_1.obj scale=0.001 0.001 0.001; visual mesh filename=k3lso/obj/thigh_hr_1.obj scale=0.001 0.001 0.001
- link thigh_hr_2: geometry collision mesh filename=k3lso/obj/thigh_hr_2.obj scale=0.001 0.001 0.001; visual mesh filename=k3lso/obj/thigh_hr_2.obj scale=0.001 0.001 0.001
- link toe_hr_1: geometry collision mesh filename=k3lso/obj/toe_hr_1.obj scale=0.001 0.001 0.001; visual mesh filename=k3lso/obj/toe_hr_1.obj scale=0.001 0.001 0.001
- link toe_hr_2: geometry collision mesh filename=k3lso/obj/toe_hr_2.obj scale=0.001 0.001 0.001; visual mesh filename=k3lso/obj/toe_hr_2.obj scale=0.001 0.001 0.001
- link toe_hr_3: geometry collision mesh filename=k3lso/obj/toe_hr_3.obj scale=0.001 0.001 0.001; visual mesh filename=k3lso/obj/toe_hr_3.obj scale=0.001 0.001 0.001
- link toe_hr_4: geometry collision mesh filename=k3lso/obj/toe_hr_4.obj scale=0.001 0.001 0.001; visual mesh filename=k3lso/obj/toe_hr_4.obj scale=0.001 0.001 0.001

Commit message: create model

File: robot_gym/util/pybullet_data/robots/k3lso.urdf (robot description, URDF)
Before this commit: robot k3lso_robot, 17 links, 16 joints
Links:
- link abduct_hr_1: geometry collision mesh filename=k3lso/obj/abduct_hr_1.obj scale=0.001 0.001 0.001; visual mesh filename=k3lso/obj/abduct_hr_1.obj scale=0.001 0.001 0.001
Joints:
- removed joint toe_fl_joint
- removed joint toe_fr_joint
- removed joint toe_hl_joint
- removed joint toe_hr_joint
- added joint fl_joint_toe: type fixed, parent shank_hl_2, child toe_hr_2, origin xyz=0.002252 -0.0177 -0.272251 rpy=0 0 0
- added joint fr_joint_toe: type fixed, parent shank_hl_1, child toe_hr_1, origin xyz=0.002252 0.0177 -0.272251 rpy=0 0 0
- added joint hl_joint_toe: type fixed, parent shank_hl_4, child toe_hr_4, origin xyz=0.002251 -0.0177 -0.272251 rpy=0 0 0
- added joint hr_joint_toe: type fixed, parent shank_hl_3, child toe_hr_3, origin xyz=0.002251 0.0177 -0.272251 rpy=0 0 0

Commit message: mods
Updating some params

File: robot_gym/util/pybullet_data/robots/k3lso.urdf (robot description, URDF)
Before this commit: robot k3lso_robot, 17 links, 16 joints
Joints:
- joint abduct_fl_to_thigh_fl_j: limit (none) -> effort=54 velocity=100
- joint abduct_fr_to_thigh_fr_j: limit (none) -> effort=54 velocity=100
- joint abduct_hl_to_thigh_hl_j: limit (none) -> effort=54 velocity=100
- joint abduct_hr_to_thigh_hr_j: limit (none) -> effort=54 velocity=100
- joint thigh_fl_to_knee_fl_j: limit (none) -> effort=54 velocity=100
- joint thigh_fr_to_knee_fr_j: limit (none) -> effort=54 velocity=100
- joint thigh_hl_to_knee_hl_j: limit (none) -> effort=54 velocity=100
- joint thigh_hr_to_knee_hr_j: limit (none) -> effort=54 velocity=100
- joint torso_to_abduct_fl_j: limit (none) -> effort=54 velocity=100
- joint torso_to_abduct_fr_j: limit (none) -> effort=54 velocity=100
- joint torso_to_abduct_hl_j: limit (none) -> effort=54 velocity=100
- joint torso_to_abduct_hr_j: limit (none) -> effort=54 velocity=100
