Commit message: edit go-to action space

File: robot_gym/util/pybullet_data/robots/ghost.urdf (robot description, URDF)
Before this commit: robot rex, 17 links, 16 joints
Links:
- link FL_hip: geometry collision mesh filename=ghost/hip.obj scale=1 1 1; visual mesh filename=ghost/hip.obj scale=1 1 1
- link FL_lower: geometry collision mesh filename=ghost/lower_leg.obj scale=1 1 1; visual mesh filename=ghost/lower_leg.obj scale=1 1 1
- link FL_upper: geometry collision mesh filename=ghost/upper_leg.obj scale=1 1 1; visual mesh filename=ghost/upper_leg.obj scale=1 1 1
- link FR_hip: geometry collision mesh filename=ghost/hip.obj scale=1 1 1; visual mesh filename=ghost/hip.obj scale=1 1 1
- link FR_lower: geometry collision mesh filename=ghost/lower_leg.obj scale=1 1 1; visual mesh filename=ghost/lower_leg.obj scale=1 1 1
- link FR_upper: geometry collision mesh filename=ghost/upper_leg_mirror.obj scale=1 1 1; visual mesh filename=ghost/upper_leg_mirror.obj scale=1 1 1
- link RL_hip: geometry collision mesh filename=ghost/hip.obj scale=1 1 1; visual mesh filename=ghost/hip.obj scale=1 1 1
- link RL_lower: geometry collision mesh filename=ghost/lower_leg.obj scale=1 1 1; visual mesh filename=ghost/lower_leg.obj scale=1 1 1
- link RL_upper: geometry collision mesh filename=ghost/upper_leg.obj scale=1 1 1; visual mesh filename=ghost/upper_leg.obj scale=1 1 1
- link RR_hip: geometry collision mesh filename=ghost/hip.obj scale=1 1 1; visual mesh filename=ghost/hip.obj scale=1 1 1
- link RR_lower: geometry collision mesh filename=ghost/lower_leg.obj scale=1 1 1; visual mesh filename=ghost/lower_leg.obj scale=1 1 1
- link RR_upper: geometry collision mesh filename=ghost/upper_leg_mirror.obj scale=1 1 1; visual mesh filename=ghost/upper_leg_mirror.obj scale=1 1 1
- link trunk: geometry collision mesh filename=ghost/body.obj scale=1 1 1; visual mesh filename=ghost/body.obj scale=1 1 1

Commit message: add arm model

File: robot_gym/util/pybullet_data/robots/ghost.urdf (robot description, URDF)
Before this commit: robot ghost, 17 links, 16 joints
Links:
- added link Arm_1_v1_1, mass 4.3410244605972785; collision mesh filename=spot_arm/Arm_1_v1_1.stl scale=0.001 0.001 0.001; visual mesh filename=spot_arm/Arm_1_v1_1.stl scale=0.001 0.001 0.001
- added link Arm_2_v1_1, mass 4.446518989183043; collision mesh filename=spot_arm/Arm_2_v1_1.stl scale=0.001 0.001 0.001; visual mesh filename=spot_arm/Arm_2_v1_1.stl scale=0.001 0.001 0.001
- added link arm_base_link, mass 0.8137272025946127; collision mesh filename=spot_arm/base_link.stl scale=0.001 0.001 0.001; visual mesh filename=spot_arm/base_link.stl scale=0.001 0.001 0.001
- added link bottom_v1_1, mass 3.7768145403916407; collision mesh filename=spot_arm/bottom_v1_1.stl scale=0.001 0.001 0.001; visual mesh filename=spot_arm/bottom_v1_1.stl scale=0.001 0.001 0.001
- added link gripper_v1_1, mass 0.8080491704220107; collision mesh filename=spot_arm/gripper_v1_1.stl scale=0.001 0.001 0.001; visual mesh filename=spot_arm/gripper_v1_1.stl scale=0.001 0.001 0.001
- added link head_v1_1, mass 1.2644309089007917; collision mesh filename=spot_arm/head_v1_1.stl scale=0.001 0.001 0.001; visual mesh filename=spot_arm/head_v1_1.stl scale=0.001 0.001 0.001
- added link neck_v1_1, mass 0.8026625496929148; collision mesh filename=spot_arm/neck_v1_1.stl scale=0.001 0.001 0.001; visual mesh filename=spot_arm/neck_v1_1.stl scale=0.001 0.001 0.001
Joints:
- added joint Rev1: type continuous, parent arm_base_link, child bottom_v1_1, origin xyz=0.009381 0.055159 -0.00311 rpy=0 0 0, axis 0.0 0.0 -1.0
- added joint Rev2: type continuous, parent bottom_v1_1, child Arm_1_v1_1, origin xyz=0.0315 0.0 0.0499 rpy=0 0 0, axis 1.0 -0.0 -0.0
- added joint Rev3: type continuous, parent Arm_1_v1_1, child Arm_2_v1_1, origin xyz=0.0074 0.266 0.0 rpy=0 0 0, axis -1.0 0.0 -0.0
- added joint Rev4: type continuous, parent Arm_2_v1_1, child neck_v1_1, origin xyz=-0.05805 -0.299861 0.073345 rpy=0 0 0, axis 1.0 0.0 0.0
- added joint Rev5: type continuous, parent neck_v1_1, child head_v1_1, origin xyz=0.019139 -0.04916 0.004301 rpy=0 0 0, axis -0.0 -0.996195 0.087156
- added joint Rev6: type continuous, parent head_v1_1, child gripper_v1_1, origin xyz=0.035007 -0.079919 0.021947 rpy=0 0 0, axis -1.0 0.0 -0.0
- added joint arm_base: type fixed, parent trunk, child arm_base_link, origin xyz=0 -0.057 0.13 rpy=0 0 0

Commit message: add new ghost urdf

File: robot_gym/util/pybullet_data/robots/ghost.urdf (robot description, URDF)
Before this commit: robot ghost, 24 links, 23 joints
Links:
- removed link Arm_1_v1_1
- removed link Arm_2_v1_1
- removed link bottom_v1_1
- removed link gripper_v1_1
- removed link head_v1_1
- removed link neck_v1_1
- added link arm_gripper, mass 0.8080491704220107; collision mesh filename=spot_arm/gripper_v1_1.stl scale=0.001 0.001 0.001; visual mesh filename=spot_arm/gripper_v1_1.stl scale=0.001 0.001 0.001
- added link arm_link_1, mass 3.7768145403916407; collision mesh filename=spot_arm/bottom_v1_1.stl scale=0.001 0.001 0.001; visual mesh filename=spot_arm/bottom_v1_1.stl scale=0.001 0.001 0.001
- added link arm_link_2, mass 4.3410244605972785; collision mesh filename=spot_arm/Arm_1_v1_1.stl scale=0.001 0.001 0.001; visual mesh filename=spot_arm/Arm_1_v1_1.stl scale=0.001 0.001 0.001
- added link arm_link_3, mass 4.446518989183043; collision mesh filename=spot_arm/Arm_2_v1_1.stl scale=0.001 0.001 0.001; visual mesh filename=spot_arm/Arm_2_v1_1.stl scale=0.001 0.001 0.001
- added link arm_link_4, mass 0.8026625496929148; collision mesh filename=spot_arm/neck_v1_1.stl scale=0.001 0.001 0.001; visual mesh filename=spot_arm/neck_v1_1.stl scale=0.001 0.001 0.001
- added link arm_link_5, mass 1.2644309089007917; collision mesh filename=spot_arm/head_v1_1.stl scale=0.001 0.001 0.001; visual mesh filename=spot_arm/head_v1_1.stl scale=0.001 0.001 0.001
Joints:
- removed joint Rev1
- removed joint Rev2
- removed joint Rev3
- removed joint Rev4
- removed joint Rev5
- removed joint Rev6
- added joint motor_arm_0: type continuous, parent arm_base_link, child arm_link_1, origin xyz=0.009381 0.055159 -0.00311 rpy=0 0 0, axis 0.0 0.0 -1.0
- added joint motor_arm_1: type continuous, parent arm_link_1, child arm_link_2, origin xyz=0.0315 0.0 0.0499 rpy=0 0 0, axis 1.0 -0.0 -0.0
- added joint motor_arm_2: type continuous, parent arm_link_2, child arm_link_3, origin xyz=0.0074 0.266 0.0 rpy=0 0 0, axis -1.0 0.0 -0.0
- added joint motor_arm_3: type continuous, parent arm_link_3, child arm_link_4, origin xyz=-0.05805 -0.299861 0.073345 rpy=0 0 0, axis 1.0 0.0 0.0
- added joint motor_arm_4: type continuous, parent arm_link_4, child arm_link_5, origin xyz=0.019139 -0.04916 0.004301 rpy=0 0 0, axis -0.0 -0.996195 0.087156
- added joint motor_arm_5: type continuous, parent arm_link_5, child arm_gripper, origin xyz=0.035007 -0.079919 0.021947 rpy=0 0 0, axis -1.0 0.0 -0.0

Commit message: light arm

File: robot_gym/util/pybullet_data/robots/ghost.urdf (robot description, URDF)
Before this commit: robot ghost, 24 links, 23 joints
Links:
- link arm_base_link: mass 0.8137272025946127 -> 0.5
- link arm_gripper: mass 0.8080491704220107 -> 1
- link arm_link_1: mass 3.7768145403916407 -> 0.5
- link arm_link_2: mass 4.3410244605972785 -> 0.5
- link arm_link_3: mass 4.446518989183043 -> 0.5
- link arm_link_4: mass 0.8026625496929148 -> 0.5
- link arm_link_5: mass 1.2644309089007917 -> 0.5

Commit message: Add amber_b1 arm

File: robot_gym/util/pybullet_data/robots/ghost.urdf (robot description, URDF)
Before this commit: robot ghost, 24 links, 23 joints
Links:
- removed link arm_gripper
- removed link arm_link_1
- removed link arm_link_2
- removed link arm_link_3
- removed link arm_link_4
- removed link arm_link_5
- added link DOF1_1, mass 0.6510136315044379; collision mesh filename=amber_b1/DOF1_1.stl scale=0.001 0.001 0.001; visual mesh filename=amber_b1/DOF1_1.stl scale=0.001 0.001 0.001
- added link DOF1_LINK_1, mass 0.935292940405524; collision mesh filename=amber_b1/DOF1_LINK_1.stl scale=0.001 0.001 0.001; visual mesh filename=amber_b1/DOF1_LINK_1.stl scale=0.001 0.001 0.001
- added link DOF2_1, mass 0.5984706718739643; collision mesh filename=amber_b1/DOF2_1.stl scale=0.001 0.001 0.001; visual mesh filename=amber_b1/DOF2_1.stl scale=0.001 0.001 0.001
- added link DOF3_LINK_1, mass 0.935292940405524; collision mesh filename=amber_b1/DOF3_LINK_1.stl scale=0.001 0.001 0.001; visual mesh filename=amber_b1/DOF3_LINK_1.stl scale=0.001 0.001 0.001
- added link DOF3_MOTOR_1, mass 0.5847003223149023; collision mesh filename=amber_b1/DOF3_MOTOR_1.stl scale=0.001 0.001 0.001; visual mesh filename=amber_b1/DOF3_MOTOR_1.stl scale=0.001 0.001 0.001
- added link DOF4_1, mass 0.5984706718739643; collision mesh filename=amber_b1/DOF4_1.stl scale=0.001 0.001 0.001; visual mesh filename=amber_b1/DOF4_1.stl scale=0.001 0.001 0.001
- added link DOF5_MOTOR_1, mass 0.5847003223149023; collision mesh filename=amber_b1/DOF5_MOTOR_1.stl scale=0.001 0.001 0.001; visual mesh filename=amber_b1/DOF5_MOTOR_1.stl scale=0.001 0.001 0.001
- added link DOF5_link_1, mass 0.935292940405524; collision mesh filename=amber_b1/DOF5_link_1.stl scale=0.001 0.001 0.001; visual mesh filename=amber_b1/DOF5_link_1.stl scale=0.001 0.001 0.001
- added link DOF6_LINK_1, mass 0.5984706718739643; collision mesh filename=amber_b1/DOF6_LINK_1.stl scale=0.001 0.001 0.001; visual mesh filename=amber_b1/DOF6_LINK_1.stl scale=0.001 0.001 0.001
- added link DOF7_MOTOR_1, mass 0.5847003223149023; collision mesh filename=amber_b1/DOF7_MOTOR_1.stl scale=0.001 0.001 0.001; visual mesh filename=amber_b1/DOF7_MOTOR_1.stl scale=0.001 0.001 0.001
- added link TOP_1, mass 0.15302388632599126; collision mesh filename=amber_b1/TOP_1.stl scale=0.001 0.001 0.001; visual mesh filename=amber_b1/TOP_1.stl scale=0.001 0.001 0.001
- link arm_base_link: mass 0.5 -> 0.28897197894505794; geometry collision mesh filename=amber_b1/base_link.stl scale=0.001 0.001 0.001; visual mesh filename=amber_b1/base_link.stl scale=0.001 0.001 0.001
Joints:
- added joint Rigid1: type fixed, parent arm_base_link, child DOF1_1, origin xyz=0.0 4e-06 0.069966 rpy=0 0 0
- added joint Rigid11: type fixed, parent DOF6_LINK_1, child DOF7_MOTOR_1, origin xyz=-0.0 0.0255 0.122896 rpy=0 0 0
- added joint Rigid12: type fixed, parent DOF6_LINK_1, child TOP_1, origin xyz=-0.0 0.0255 0.127896 rpy=0 0 0
- added joint Rigid5: type fixed, parent DOF2_1, child DOF3_MOTOR_1, origin xyz=0.0 0.0255 0.122897 rpy=0 0 0
- added joint Rigid8: type fixed, parent DOF4_1, child DOF5_MOTOR_1, origin xyz=0.0 -0.0255 0.122896 rpy=0 0 0
- joint arm_base: origin xyz=0 -0.057 0.13 rpy=0 0 0 -> xyz=0 0 0 rpy=0 0 0
- joint motor_arm_0: axis 0.0 0.0 -1.0 -> 0.0 0.0 1.0; child arm_link_1 -> DOF1_LINK_1; origin xyz=0.009381 0.055159 -0.00311 rpy=0 0 0 -> xyz=0.0 4e-06 0.074366 rpy=0 0 0
- joint motor_arm_1: axis 1.0 -0.0 -0.0 -> 0.0 1.0 -0.0; child arm_link_2 -> DOF2_1; origin xyz=0.0315 0.0 0.0499 rpy=0 0 0 -> xyz=-0.0 -0.025 0.0812 rpy=0 0 0; parent arm_link_1 -> DOF1_LINK_1
- joint motor_arm_2: axis -1.0 0.0 -0.0 -> 0.0 -0.0 -1.0; child arm_link_3 -> DOF3_LINK_1; origin xyz=0.0074 0.266 0.0 rpy=0 0 0 -> xyz=0.0 0.0255 0.127897 rpy=0 0 0; parent arm_link_2 -> DOF2_1
- joint motor_arm_3: axis 1.0 0.0 0.0 -> 0.0 -1.0 -0.0; child arm_link_4 -> DOF4_1; origin xyz=-0.05805 -0.299861 0.073345 rpy=0 0 0 -> xyz=0.0 0.025 0.0815 rpy=0 0 0; parent arm_link_3 -> DOF3_LINK_1
- joint motor_arm_4: axis -0.0 -0.996195 0.087156 -> -0.0 0.0 -1.0; child arm_link_5 -> DOF5_link_1; origin xyz=0.019139 -0.04916 0.004301 rpy=0 0 0 -> xyz=0.0 -0.0255 0.127896 rpy=0 0 0; parent arm_link_4 -> DOF4_1
- joint motor_arm_5: axis -1.0 0.0 -0.0 -> 0.0 1.0 0.0; child arm_gripper -> DOF6_LINK_1; origin xyz=0.035007 -0.079919 0.021947 rpy=0 0 0 -> xyz=0.0 -0.025 0.0812 rpy=0 0 0; parent arm_link_5 -> DOF5_link_1

File: robot_gym/util/pybullet_data/robots/k3lso.urdf (robot description, URDF)
Before this commit: robot k3lso_robot, 17 links, 16 joints
Links:
- added link DOF1_1, mass 0.6510136315044379; collision mesh filename=amber_b1/DOF1_1.stl scale=0.001 0.001 0.001; visual mesh filename=amber_b1/DOF1_1.stl scale=0.001 0.001 0.001
- added link DOF1_LINK_1, mass 0.935292940405524; collision mesh filename=amber_b1/DOF1_LINK_1.stl scale=0.001 0.001 0.001; visual mesh filename=amber_b1/DOF1_LINK_1.stl scale=0.001 0.001 0.001
- added link DOF2_1, mass 0.5984706718739643; collision mesh filename=amber_b1/DOF2_1.stl scale=0.001 0.001 0.001; visual mesh filename=amber_b1/DOF2_1.stl scale=0.001 0.001 0.001
- added link DOF3_LINK_1, mass 0.935292940405524; collision mesh filename=amber_b1/DOF3_LINK_1.stl scale=0.001 0.001 0.001; visual mesh filename=amber_b1/DOF3_LINK_1.stl scale=0.001 0.001 0.001
- added link DOF3_MOTOR_1, mass 0.5847003223149023; collision mesh filename=amber_b1/DOF3_MOTOR_1.stl scale=0.001 0.001 0.001; visual mesh filename=amber_b1/DOF3_MOTOR_1.stl scale=0.001 0.001 0.001
- added link DOF4_1, mass 0.5984706718739643; collision mesh filename=amber_b1/DOF4_1.stl scale=0.001 0.001 0.001; visual mesh filename=amber_b1/DOF4_1.stl scale=0.001 0.001 0.001
- added link DOF5_MOTOR_1, mass 0.5847003223149023; collision mesh filename=amber_b1/DOF5_MOTOR_1.stl scale=0.001 0.001 0.001; visual mesh filename=amber_b1/DOF5_MOTOR_1.stl scale=0.001 0.001 0.001
- added link DOF5_link_1, mass 0.935292940405524; collision mesh filename=amber_b1/DOF5_link_1.stl scale=0.001 0.001 0.001; visual mesh filename=amber_b1/DOF5_link_1.stl scale=0.001 0.001 0.001
- added link DOF6_LINK_1, mass 0.5984706718739643; collision mesh filename=amber_b1/DOF6_LINK_1.stl scale=0.001 0.001 0.001; visual mesh filename=amber_b1/DOF6_LINK_1.stl scale=0.001 0.001 0.001
- added link DOF7_MOTOR_1, mass 0.5847003223149023; collision mesh filename=amber_b1/DOF7_MOTOR_1.stl scale=0.001 0.001 0.001; visual mesh filename=amber_b1/DOF7_MOTOR_1.stl scale=0.001 0.001 0.001
- added link TOP_1, mass 0.15302388632599126; collision mesh filename=amber_b1/TOP_1.stl scale=0.001 0.001 0.001; visual mesh filename=amber_b1/TOP_1.stl scale=0.001 0.001 0.001
- added link arm_base_link, mass 0.28897197894505794; collision mesh filename=amber_b1/base_link.stl scale=0.001 0.001 0.001; visual mesh filename=amber_b1/base_link.stl scale=0.001 0.001 0.001
Joints:
- added joint Rigid1: type fixed, parent arm_base_link, child DOF1_1, origin xyz=0.0 4e-06 0.069966 rpy=0 0 0
- added joint Rigid11: type fixed, parent DOF6_LINK_1, child DOF7_MOTOR_1, origin xyz=-0.0 0.0255 0.122896 rpy=0 0 0
- added joint Rigid12: type fixed, parent DOF6_LINK_1, child TOP_1, origin xyz=-0.0 0.0255 0.127896 rpy=0 0 0
- added joint Rigid5: type fixed, parent DOF2_1, child DOF3_MOTOR_1, origin xyz=0.0 0.0255 0.122897 rpy=0 0 0
- added joint Rigid8: type fixed, parent DOF4_1, child DOF5_MOTOR_1, origin xyz=0.0 -0.0255 0.122896 rpy=0 0 0
- added joint arm_base: type fixed, parent base_link, child arm_base_link, origin xyz=0 0 0 rpy=0 0 0
- added joint motor_arm_0: type continuous, parent arm_base_link, child DOF1_LINK_1, origin xyz=0.0 4e-06 0.074366 rpy=0 0 0, axis 0.0 0.0 1.0
- added joint motor_arm_1: type continuous, parent DOF1_LINK_1, child DOF2_1, origin xyz=-0.0 -0.025 0.0812 rpy=0 0 0, axis 0.0 1.0 -0.0
- added joint motor_arm_2: type continuous, parent DOF2_1, child DOF3_LINK_1, origin xyz=0.0 0.0255 0.127897 rpy=0 0 0, axis 0.0 -0.0 -1.0
- added joint motor_arm_3: type continuous, parent DOF3_LINK_1, child DOF4_1, origin xyz=0.0 0.025 0.0815 rpy=0 0 0, axis 0.0 -1.0 -0.0
- added joint motor_arm_4: type continuous, parent DOF4_1, child DOF5_link_1, origin xyz=0.0 -0.0255 0.127896 rpy=0 0 0, axis -0.0 0.0 -1.0
- added joint motor_arm_5: type continuous, parent DOF5_link_1, child DOF6_LINK_1, origin xyz=0.0 -0.025 0.0812 rpy=0 0 0, axis 0.0 1.0 0.0

Commit message: Spot Arm Mini

File: robot_gym/util/pybullet_data/robots/ghost.urdf (robot description, URDF)
Before this commit: robot ghost, 29 links, 28 joints
Links:
- removed link DOF1_1
- removed link DOF1_LINK_1
- removed link DOF2_1
- removed link DOF3_LINK_1
- removed link DOF3_MOTOR_1
- removed link DOF4_1
- removed link DOF5_MOTOR_1
- removed link DOF5_link_1
- removed link DOF6_LINK_1
- removed link DOF7_MOTOR_1
- removed link TOP_1
- added link arm_gripper, mass 1.5302388632599126; collision mesh filename=spot_arm/gripper_v1_1.stl; visual mesh filename=spot_arm/gripper_v1_1.stl
- added link arm_link_1, mass 0.6510136315044379; collision mesh filename=spot_arm/bottom_v1_1.stl; visual mesh filename=spot_arm/bottom_v1_1.stl
- added link arm_link_2, mass 1.935292940405524; collision mesh filename=spot_arm/Arm_1_v1_1.stl; visual mesh filename=spot_arm/Arm_1_v1_1.stl
- added link arm_link_3, mass 1.935292940405524; collision mesh filename=spot_arm/Arm_2_v1_1.stl; visual mesh filename=spot_arm/Arm_2_v1_1.stl
- added link arm_link_4, mass 1.935292940405524; collision mesh filename=spot_arm/neck_v1_1.stl; visual mesh filename=spot_arm/neck_v1_1.stl
- added link arm_link_5, mass 0.28897197894505794; collision mesh filename=spot_arm/head_v1_1.stl; visual mesh filename=spot_arm/head_v1_1.stl
- link arm_base_link: geometry collision mesh filename=spot_arm/base_link.stl; visual mesh filename=spot_arm/base_link.stl
Joints:
- removed joint Rigid1
- removed joint Rigid11
- removed joint Rigid12
- removed joint Rigid5
- removed joint Rigid8
- joint arm_base: origin xyz=0 0 0 rpy=0 0 0 -> xyz=0 0 0.1 rpy=0 0 0
- joint motor_arm_0: axis 0.0 0.0 1.0 -> 0.0 0.0 -1.0; child DOF1_LINK_1 -> arm_link_1; origin xyz=0.0 4e-06 0.074366 rpy=0 0 0 -> xyz=0.0 0.002 0.046 rpy=0 0 0
- joint motor_arm_1: axis 0.0 1.0 -0.0 -> 1.0 -0.0 -0.0; child DOF2_1 -> arm_link_2; origin xyz=-0.0 -0.025 0.0812 rpy=0 0 0 -> xyz=0.0 0.0 0.0 rpy=0 0 0; parent DOF1_LINK_1 -> arm_link_1
- joint motor_arm_2: axis 0.0 -0.0 -1.0 -> -1.0 0.0 -0.0; child DOF3_LINK_1 -> arm_link_3; origin xyz=0.0 0.0255 0.127897 rpy=0 0 0 -> xyz=-0.0015 0.21 0 rpy=0 0 0; parent DOF2_1 -> arm_link_2
- joint motor_arm_3: axis 0.0 -1.0 -0.0 -> 1.0 0.0 0.0; child DOF4_1 -> arm_link_4; origin xyz=0.0 0.025 0.0815 rpy=0 0 0 -> xyz=0 -0.24 0.06 rpy=0 0 0; parent DOF3_LINK_1 -> arm_link_3
- joint motor_arm_4: axis -0.0 0.0 -1.0 -> -0.0 -1.0 0.0; child DOF5_link_1 -> arm_link_5; origin xyz=0.0 -0.0255 0.127896 rpy=0 0 0 -> xyz=0 -0.045 0 rpy=0 0 0; parent DOF4_1 -> arm_link_4
- joint motor_arm_5: axis 0.0 1.0 0.0 -> -1.0 0.0 -0.0; child DOF6_LINK_1 -> arm_gripper; origin xyz=0.0 -0.025 0.0812 rpy=0 0 0 -> xyz=0.002 -0.04 0.015 rpy=0 0 0; parent DOF5_link_1 -> arm_link_5

Commit message: igibson base integration (beta)

File: robot_gym/util/pybullet_data/robots/ghost.urdf (robot description, URDF)
Before this commit: robot ghost, 24 links, 23 joints
Links:
- removed link trunk
- added link base_link, mass 13.715; collision mesh filename=ghost/body.obj scale=1 1 1; visual mesh filename=ghost/body.obj scale=1 1 1
- added link eyes, mass 0.001
- added link laser_link, mass 0.00833634573995571; collision mesh filename=laser/laser_link.obj; visual mesh filename=laser/laser_link.obj
Joints:
- added joint eye_joint: type fixed, parent base_link, child eyes, origin xyz=0.1 0 0.1 rpy=0 0 0
- added joint laser_joint: type fixed, parent base_link, child laser_link, origin xyz=0.0 0 -0.1 rpy=3.14159265359 0 0, axis 0 0 0
- joint FL_hip_joint: parent trunk -> base_link
- joint FR_hip_joint: parent trunk -> base_link
- joint RL_hip_joint: parent trunk -> base_link
- joint RR_hip_joint: parent trunk -> base_link
- joint arm_base: parent trunk -> base_link
